File: hardware/SmartNerfBlaster-v1/SmartNerfBlaster.sch (KiCad schematic (older format))
At the start: 34 parts, among them J1 Conn_01x02_Male, J2 Conn_01x06_Male, J3 Conn_01x04_Male, J4 Screw_Terminal_01x02, J5 Screw_Terminal_01x02, J6 Conn_02x03_Odd_Even, Q1 FQP30N06L, Q2 FQP30N06L, U1 L7805, U2 ATmega328P-PU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

Commit message: Fixed libaray issues. Added gerbers and pdf outputs.
Parts:
- Q1, Q2: symbol SmartNerfBlaster-rescue:FQP30N06L-SmartNerfBlasterSymbols -> SmartNerfBlasterSymbols:FQP30N06L
Other:
- moved on the sheet: D1, D2, D3, R10, R11, R9
Changed lines of the file:
@@
 EELAYER 26 0
 EELAYER END
-$Descr A4 11693 8268
+$Descr USLetter 11000 8500
 encoding utf-8
 Sheet 1 1
-Title ""
-Date ""
-Rev ""
-Comp ""
-Comment1 ""
+Title "SmartNerfBlaster"
+Date "2019-03-04"
+Rev "v1"
+Comp "Dan Kirkham"
+Comment1 "github.com/dankirkham"
 Comment2 ""
 Comment3 ""
@@
 L Device:LED D1
 U 1 1 5C72AE44
-P 9500 2350
-F 0 "D1" V 9538 2233 50  0000 R CNN
-F 1 "LED" V 9447 2233 50  0000 R CNN
-F 2 "LEDs:LED_D3.0mm" H 9500 2350 50  0001 C CNN
-F 3 "~" H 9500 2350 50  0001 C CNN
-	1    9500 2350
+P 8800 1950
+F 0 "D1" V 8838 1833 50  0000 R CNN
+F 1 "LED" V 8747 1833 50  0000 R CNN
+F 2 "LEDs:LED_D3.0mm" H 8800 1950 50  0001 C CNN
+F 3 "~" H 8800 1950 50  0001 C CNN
+	1    8800 1950
 	0    -1   -1   0
 $EndComp
@@
 L Device:LED D2
 U 1 1 5C72AF00
-P 9900 2350
-F 0 "D2" V 9938 2233 50  0000 R CNN
-F 1 "LED" V 9847 2233 50  0000 R CNN
-F 2 "LEDs:LED_D3.0mm" H 9900 2350 50  0001 C CNN
-F 3 "~" H 9900 2350 50  0001 C CNN
-	1    9900 2350
+P 9200 1950
+F 0 "D2" V 9238 1833 50  0000 R CNN
+F 1 "LED" V 9147 1833 50  0000 R CNN
+F 2 "LEDs:LED_D3.0mm" H 9200 1950 50  0001 C CNN
+F 3 "~" H 9200 1950 50  0001 C CNN
+	1    9200 1950
 	0    -1   -1   0
 $EndComp
@@
 L Device:LED D3
 U 1 1 5C72AF4F
-P 10300 2350
-F 0 "D3" V 10338 2233 50  0000 R CNN
-F 1 "LED" V 10247 2233 50  0000 R CNN
-F 2 "LEDs:LED_D3.0mm" H 10300 2350 50  0001 C CNN
-F 3 "~" H 10300 2350 50  0001 C CNN
-	1    10300 2350
+P 9600 1950
+F 0 "D3" V 9638 1833 50  0000 R CNN
+F 1 "LED" V 9547 1833 50  0000 R CNN
+F 2 "LEDs:LED_D3.0mm" H 9600 1950 50  0001 C CNN
+F 3 "~" H 9600 1950 50  0001 C CNN
+	1    9600 1950
 	0    -1   -1   0
 $EndComp
-Text Label 9500 2000 0    50   ~ 0
+Text Label 8800 1600 0    50   ~ 0
 LED1
-Text Label 9900 2000 0    50   ~ 0
+Text Label 9200 1600 0    50   ~ 0
 LED2
-Text Label 10300 2000 0    50   ~ 0
+Text Label 9600 1600 0    50   ~ 0
 LED3
 $Comp
 L Device:R R9
 U 1 1 5C72B2C1
-P 9500 2850
-F 0 "R9" H 9570 2896 50  0000 L CNN
-F 1 "330" H 9570 2805 50  0000 L CNN
-F 2 "Resistors_THT:R_Axial_DIN0207_L6.3mm_D2.5mm_P2.54mm_Vertical" V 9430 2850 50  0001 C CNN
-F 3 "~" H 9500 2850 50  0001 C CNN
-	1    9500 2850
+P 8800 2450
+F 0 "R9" H 8870 2496 50  0000 L CNN
+F 1 "330" H 8870 2405 50  0000 L CNN
+F 2 "Resistors_THT:R_Axial_DIN0207_L6.3mm_D2.5mm_P2.54mm_Vertical" V 8730 2450 50  0001 C CNN
+F 3 "~" H 8800 2450 50  0001 C CNN
+	1    8800 2450
 	1    0    0    -1
 $EndComp
@@
 L Device:R R10
 U 1 1 5C72B357
-P 9900 2850
-F 0 "R10" H 9970 2896 50  0000 L CNN
-F 1 "330" H 9970 2805 50  0000 L CNN
-F 2 "Resistors_THT:R_Axial_DIN0207_L6.3mm_D2.5mm_P2.54mm_Vertical" V 9830 2850 50  0001 C CNN
-F 3 "~" H 9900 2850 50  0001 C CNN
-	1    9900 2850
+P 9200 2450
+F 0 "R10" H 9270 2496 50  0000 L CNN
+F 1 "330" H 9270 2405 50  0000 L CNN
+F 2 "Resistors_THT:R_Axial_DIN0207_L6.3mm_D2.5mm_P2.54mm_Vertical" V 9130 2450 50  0001 C CNN
+F 3 "~" H 9200 2450 50  0001 C CNN
+	1    9200 2450
 	1    0    0    -1
 $EndComp
@@
 L Device:R R11
 U 1 1 5C72B3EB
-P 10300 2850
-F 0 "R11" H 10370 2896 50  0000 L CNN
-F 1 "330" H 10370 2805 50  0000 L CNN
-F 2 "Resistors_THT:R_Axial_DIN0207_L6.3mm_D2.5mm_P2.54mm_Vertical" V 10230 2850 50  0001 C CNN
-F 3 "~" H 10300 2850 50  0001 C CNN
-	1    10300 2850
-	1    0    0    -1
-$EndComp
-Wire Wire Line
-	9500 2500 9500 2700
-Wire Wire Line
-	9500 2200 9500 2000
-Wire Wire Line
-	9900 2000 9900 2200
-Wire Wire Line
-	10300 2000 10300 2200
-Wire Wire Line
-	10300 2500 10300 2700
-Wire Wire Line
-	9900 2500 9900 2700
+P 9600 2450
+F 0 "R11" H 9670 2496 50  0000 L CNN
+F 1 "330" H 9670 2405 50  0000 L CNN
+F 2 "Resistors_THT:R_Axial_DIN0207_L6.3mm_D2.5mm_P2.54mm_Vertical" V 9530 2450 50  0001 C CNN
+F 3 "~" H 9600 2450 50  0001 C CNN
+	1    9600 2450
+	1    0    0    -1
+$EndComp
+Wire Wire Line
+	8800 2100 8800 2300
+Wire Wire Line
+	8800 1800 8800 1600
+Wire Wire Line
+	9200 1600 9200 1800
+Wire Wire Line
+	9600 1600 9600 1800
+Wire Wire Line
+	9600 2100 9600 2300
+Wire Wire Line
+	9200 2100 9200 2300
 $Comp
 L power:GND #PWR0125
 U 1 1 5C751B84
-P 9500 3150
-F 0 "#PWR0125" H 9500 2900 50  0001 C CNN
-F 1 "GND" H 9505 2977 50  0000 C CNN
-F 2 "" H 9500 3150 50  0001 C CNN
-F 3 "" H 9500 3150 50  0001 C CNN
-	1    9500 3150
+P 8800 2750
+F 0 "#PWR0125" H 8800 2500 50  0001 C CNN
+F 1 "GND" H 8805 2577 50  0000 C CNN
+F 2 "" H 8800 2750 50  0001 C CNN
+F 3 "" H 8800 2750 50  0001 C CNN
+	1    8800 2750
 	1    0    0    -1
 $EndComp
@@
 L power:GND #PWR0126
 U 1 1 5C751C79
-P 9900 3150
-F 0 "#PWR0126" H 9900 2900 50  0001 C CNN
-F 1 "GND" H 9905 2977 50  0000 C CNN
-F 2 "" H 9900 3150 50  0001 C CNN
-F 3 "" H 9900 3150 50  0001 C CNN
-	1    9900 3150
+P 9200 2750
+F 0 "#PWR0126" H 9200 2500 50  0001 C CNN
+F 1 "GND" H 9205 2577 50  0000 C CNN
+F 2 "" H 9200 2750 50  0001 C CNN
+F 3 "" H 9200 2750 50  0001 C CNN
+	1    9200 2750
 	1    0    0    -1
 $EndComp
@@
 L power:GND #PWR0127
 U 1 1 5C751D08
-P 10300 3150
-F 0 "#PWR0127" H 10300 2900 50  0001 C CNN
-F 1 "GND" H 10305 2977 50  0000 C CNN
-F 2 "" H 10300 3150 50  0001 C CNN
-F 3 "" H 10300 3150 50  0001 C CNN
-	1    10300 3150
-	1    0    0    -1
-$EndComp
-Wire Wire Line
-	10300 3150 10300 3000
-Wire Wire Line
-	9900 3000 9900 3150
-Wire Wire Line
-	9500 3150 9500 3000
-$Comp
-L SmartNerfBlaster-rescue:FQP30N06L-SmartNerfBlasterSymbols Q1
+P 9600 2750
+F 0 "#PWR0127" H 9600 2500 50  0001 C CNN
+F 1 "GND" H 9605 2577 50  0000 C CNN
+F 2 "" H 9600 2750 50  0001 C CNN
+F 3 "" H 9600 2750 50  0001 C CNN
+	1    9600 2750
+	1    0    0    -1
+$EndComp
+Wire Wire Line
+	9600 2750 9600 2600
+Wire Wire Line
+	9200 2600 9200 2750
+Wire Wire Line
+	8800 2750 8800 2600
+$Comp
+L SmartNerfBlasterSymbols:FQP30N06L Q1
 U 1 1 5C82A233
 P 3900 6200
@@
 $EndComp
 $Comp
-L SmartNerfBlaster-rescue:FQP30N06L-SmartNerfBlasterSymbols Q2
+L SmartNerfBlasterSymbols:FQP30N06L Q2
 U 1 1 5C82A2CE
 P 5300 6200

Commit message: Fixed more library issues.
Parts:
- J1: footprint NerfPlasterFootprints:XT-60 -> SmartNerfBlasterFootprints:XT-60
Changed lines of the file:
@@
 F 0 "J1" H 1506 2978 50  0000 C CNN
 F 1 "Conn_01x02_Male" H 1506 2887 50  0000 C CNN
-F 2 "NerfPlasterFootprints:XT-60" H 1400 2800 50  0001 C CNN
+F 2 "SmartNerfBlasterFootprints:XT-60" H 1400 2800 50  0001 C CNN
 F 3 "~" H 1400 2800 50  0001 C CNN
 	1    1400 2800
